Commit message: Change the wheels and the lidar positions so they are well positioned Also show lidar visualization and modify ranges in Gazebo

File: robot/ros_ws/src/robot_description/models/gazebo_plugins.xacro (robot description, xacro)
@@ -45,6 +45,6 @@
     <gazebo reference="lidar_link">
         <sensor name="laser" type="ray">
-            <pose> 0 0 0.3 0 0 0 </pose>
-            <visualize>false</visualize>
+            <pose> 0 0 0.0 0 0 0 </pose>
+            <visualize>true</visualize>
             <update_rate>10</update_rate>
             <ray>
@@ -57,6 +57,6 @@
                 </scan>
                 <range>
-                    <min>0.3</min>
-                    <max>12</max>
+                    <min>0.15</min>
+                    <max>4</max>
                 </range>
             </ray>

File: robot/ros_ws/src/robot_description/models/robot_core.xacro (robot description, xacro)
@@ -45,5 +45,5 @@
         </inertial>
         <visual>
-            <origin xyz="-0.018 0 0" rpy="0 0 0" />
+            <origin xyz="0 0 0" rpy="0 0 0" />
             <geometry>
                 <mesh filename="file://$(find robot_description)/meshes/left_wheel_link.STL" />
@@ -54,5 +54,5 @@
         </visual>
         <collision>
-            <origin xyz="-0.018 0 0" rpy="0 0 0" />
+            <origin xyz="0 0 0" rpy="0 0 0" />
             <geometry>
                 <mesh filename="file://$(find robot_description)/meshes/left_wheel_link.STL" />
@@ -81,5 +81,5 @@
         </inertial>
         <visual>
-            <origin xyz="-0.018 0 0" rpy="0 0 0" />
+            <origin xyz="-0.045 0 0" rpy="0 0 0" />
             <geometry>
                 <mesh filename="file://$(find robot_description)/meshes/right_wheel_link.STL" />
@@ -90,5 +90,5 @@
         </visual>
         <collision>
-            <origin xyz="0 0 0" rpy="0 0 0" />
+            <origin xyz="-0.045 0 0" rpy="0 0 0" />
             <geometry>
                 <mesh filename="file://$(find robot_description)/meshes/right_wheel_link.STL" />
