Commit message: Enable LaserScan in RVIZ
If lidar_joint type is 'continuous', there no tf for lidar_link so rviz doesn't show the lidar values

if lidar_joint type is 'fixed' and there is inertial values, the robot drifts in Gazebo

File: robot/ros_ws/src/robot_description/models/robot_core.xacro (robot description, xacro)
@@ -175,16 +175,4 @@
     </joint>
     <link name="lidar_link">
-        <inertial>
-            <origin xyz="9.9508E-08 4.832E-08 -0.015186" rpy="0 0 0" />
-            <mass value="0.041055" />
-            <inertia
-                ixx="7.8469E-06"
-                ixy="-1.4154E-11"
-                ixz="3.1419E-12"
-                iyy="7.8472E-06"
-                iyz="9.3363E-12"
-                izz="8.5515E-06"
-            />
-        </inertial>
         <visual>
             <origin xyz="0 0 0" rpy="3.1415 0 0" />
@@ -203,5 +191,5 @@
         </collision>
     </link>
-    <joint name="lidar_joint" type="continuous">
+    <joint name="lidar_joint" type="fixed">
         <origin xyz="0 0 0.383" rpy="0 0 -3.1416" />
         <parent link="base_link" />
