Commit message: Rename from robot to herminebot

File: robot/ros_ws/src/herminebot_description/models/herminebot_core.xacro (robot description, xacro)
@@ -18,5 +18,5 @@
             <origin xyz="0 0 0" rpy="-1.5708 0 3.1415" />
             <geometry>
-                <mesh filename="file://$(find robot_description)/meshes/base_link.STL" />
+                <mesh filename="file://$(find herminebot_description)/meshes/base_link.STL" />
             </geometry>
             <material name="">
@@ -27,5 +27,5 @@
             <origin xyz="0 0 0" rpy="-1.5708 0 3.1415" />
             <geometry>
-                <mesh filename="file://$(find robot_description)/meshes/base_link.STL" />
+                <mesh filename="file://$(find herminebot_description)/meshes/base_link.STL" />
             </geometry>
         </collision>
@@ -47,14 +47,14 @@
             <origin xyz="0 0 0" rpy="0 0 0" />
             <geometry>
-                <mesh filename="file://$(find robot_description)/meshes/left_wheel_link.STL" />
-            </geometry>
-            <material name="">
-                <color rgba="0.79216 0.81961 0.93333 1" />
-            </material>
-        </visual>
-        <collision>
-            <origin xyz="0 0 0" rpy="0 0 0" />
-            <geometry>
-                <mesh filename="file://$(find robot_description)/meshes/left_wheel_link.STL" />
+                <mesh filename="file://$(find herminebot_description)/meshes/left_wheel_link.STL" />
+            </geometry>
+            <material name="">
+                <color rgba="0.79216 0.81961 0.93333 1" />
+            </material>
+        </visual>
+        <collision>
+            <origin xyz="0 0 0" rpy="0 0 0" />
+            <geometry>
+                <mesh filename="file://$(find herminebot_description)/meshes/left_wheel_link.STL" />
             </geometry>
         </collision>
@@ -83,5 +83,5 @@
             <origin xyz="-0.045 0 0" rpy="0 0 0" />
             <geometry>
-                <mesh filename="file://$(find robot_description)/meshes/right_wheel_link.STL" />
+                <mesh filename="file://$(find herminebot_description)/meshes/right_wheel_link.STL" />
             </geometry>
             <material name="">
@@ -92,5 +92,5 @@
             <origin xyz="-0.045 0 0" rpy="0 0 0" />
             <geometry>
-                <mesh filename="file://$(find robot_description)/meshes/right_wheel_link.STL" />
+                <mesh filename="file://$(find herminebot_description)/meshes/right_wheel_link.STL" />
             </geometry>
         </collision>
@@ -118,5 +118,5 @@
             <origin xyz="0 0 0" rpy="1.5708 3.1415 0" />
             <geometry>
-                <mesh filename="file://$(find robot_description)/meshes/gripper_left_link.STL" />
+                <mesh filename="file://$(find herminebot_description)/meshes/gripper_left_link.STL" />
             </geometry>
             <material name="">
@@ -127,5 +127,5 @@
             <origin xyz="0 0 0" rpy="0 0 0" />
             <geometry>
-                <mesh filename="file://$(find robot_description)/meshes/gripper_left_link.STL" />
+                <mesh filename="file://$(find herminebot_description)/meshes/gripper_left_link.STL" />
             </geometry>
         </collision>
@@ -154,14 +154,14 @@
             <origin xyz="0 0 0" rpy="1.5708 3.1415 0" />
             <geometry>
-                <mesh filename="file://$(find robot_description)/meshes/gripper_right_link.STL" />
-            </geometry>
-            <material name="">
-                <color rgba="0.79216 0.81961 0.93333 1" />
-            </material>
-        </visual>
-        <collision>
-            <origin xyz="0 0 0" rpy="0 0 0" />
-            <geometry>
-                <mesh filename="file://$(find robot_description)/meshes/gripper_right_link.STL" />
+                <mesh filename="file://$(find herminebot_description)/meshes/gripper_right_link.STL" />
+            </geometry>
+            <material name="">
+                <color rgba="0.79216 0.81961 0.93333 1" />
+            </material>
+        </visual>
+        <collision>
+            <origin xyz="0 0 0" rpy="0 0 0" />
+            <geometry>
+                <mesh filename="file://$(find herminebot_description)/meshes/gripper_right_link.STL" />
             </geometry>
         </collision>
@@ -178,5 +178,5 @@
             <origin xyz="0 0 0" rpy="3.1415 0 0" />
             <geometry>
-                <mesh filename="file://$(find robot_description)/meshes/lidar_link.STL" />
+                <mesh filename="file://$(find herminebot_description)/meshes/lidar_link.STL" />
             </geometry>
             <material name="">
@@ -187,5 +187,5 @@
             <origin xyz="0 0 0" rpy="0 0 0" />
             <geometry>
-                <mesh filename="file://$(find robot_description)/meshes/lidar_link.STL" />
+                <mesh filename="file://$(find herminebot_description)/meshes/lidar_link.STL" />
             </geometry>
         </collision>
@@ -213,14 +213,14 @@
             <origin xyz="0 0 0" rpy="0 0 0" />
             <geometry>
-                <mesh filename="file://$(find robot_description)/meshes/imu_link.STL" />
-            </geometry>
-            <material name="">
-                <color rgba="0.79216 0.81961 0.93333 1" />
-            </material>
-        </visual>
-        <collision>
-            <origin xyz="0 0 0" rpy="0 0 0" />
-            <geometry>
-                <mesh filename="file://$(find robot_description)/meshes/imu_link.STL" />
+                <mesh filename="file://$(find herminebot_description)/meshes/imu_link.STL" />
+            </geometry>
+            <material name="">
+                <color rgba="0.79216 0.81961 0.93333 1" />
+            </material>
+        </visual>
+        <collision>
+            <origin xyz="0 0 0" rpy="0 0 0" />
+            <geometry>
+                <mesh filename="file://$(find herminebot_description)/meshes/imu_link.STL" />
             </geometry>
         </collision>
