Commit message: allow amcl to determine robot's pose

File: robot/ros_ws/src/herminebot_description/models/gazebo_plugins.xacro (robot description, xacro)
@@ -23,5 +23,4 @@
         <material>Gazebo/Blue</material>
     </gazebo>
-    <!-- Plugin controlleur robot differentiel -->
     <gazebo>
         <plugin name="diff_drive" filename="libgazebo_ros_diff_drive.so">
@@ -31,4 +30,5 @@
             <wheel_separation>0.297</wheel_separation> <!-- Valeur a modifier -->
             <wheel_diameter>0.06</wheel_diameter> <!-- Valeur a modifier -->
+            <command_topic>cmd_vel</command_topic>
             <!-- Limits -->
             <max_wheel_torque>200</max_wheel_torque>
@@ -38,9 +38,22 @@
             <robot_base_frame>base_link</robot_base_frame>
             <publish_odom>true</publish_odom>
-            <publish_odom_tf>true</publish_odom_tf>
-            <publish_wheel_tf>true</publish_wheel_tf>
+            <publish_odom_tf>false</publish_odom_tf>
+            <publish_wheel_tf>false</publish_wheel_tf>
+            <odometry_topic>odom</odometry_topic>
+            <odometry_frame>odom</odometry_frame>
+            <robot_base_frame>base_footprint</robot_base_frame>
+            <!-- Odometry source, 0 for ENCODER, 1 for WORLD, defaults to WORLD -->
+            <odometry_source>1</odometry_source>
             <ros>
                 <remapping>odom:=wheel/odometry</remapping>
             </ros>
+        </plugin>
+        <plugin name="herminebot_joint_state" filename="libgazebo_ros_joint_state_publisher.so">
+            <ros>
+                <remapping>~/out:=joint_states</remapping>
+            </ros>
+            <update_rate>30</update_rate>
+            <joint_name>left_wheel_joint</joint_name>
+            <joint_name>right_wheel_joint</joint_name>
         </plugin>
     </gazebo>
@@ -50,4 +63,5 @@
             <pose> 0 0 0.0 0 0 0 </pose>
             <visualize>true</visualize>
+            <always_on>true</always_on>
             <update_rate>10</update_rate>
             <ray>
@@ -81,16 +95,16 @@
             <topic>__default_topic__</topic>
             <plugin filename="libgazebo_ros_imu_sensor.so" name="imu_plugin">
-            <topicName>imu</topicName>
-            <bodyName>imu_link</bodyName>
-            <updateRateHZ>10.0</updateRateHZ>
-            <gaussianNoise>0.0</gaussianNoise>
-            <xyzOffset>0 0 0</xyzOffset>
-            <rpyOffset>0 0 0</rpyOffset>
-            <frameName>imu_link</frameName>
-            <initialOrientationAsReference>false</initialOrientationAsReference>
-            <ros>
-                  <namespace>/imu</namespace>
-                  <remapping>~/out:=data</remapping>
-            </ros>
+                <topicName>imu</topicName>
+                <bodyName>imu_link</bodyName>
+                <updateRateHZ>10.0</updateRateHZ>
+                <gaussianNoise>0.0</gaussianNoise>
+                <xyzOffset>0 0 0</xyzOffset>
+                <rpyOffset>0 0 0</rpyOffset>
+                <frameName>imu_link</frameName>
+                <initial_orientation_as_reference>false</initial_orientation_as_reference>
+                <ros>
+                      <namespace>/imu</namespace>
+                      <remapping>~/out:=data</remapping>
+                </ros>
             </plugin>
             <pose>0 0 0 0 0 0</pose>

File: robot/ros_ws/src/herminebot_description/models/herminebot_core.xacro (robot description, xacro)
@@ -2,4 +2,13 @@
 <!--suppress XmlUnusedNamespaceDeclaration -->
 <robot xmlns:xacro="http://www.ros.org/wiki/xacro" >
+    <!-- ****************** ROBOT BASE FOOTPRINT ***************************  -->
+    <!-- Define the center of the main robot chassis projected on the ground -->
+    <link name="base_footprint"/>
+    <!-- The base footprint of the robot is located underneath the chassis -->
+    <joint name="base_joint" type="fixed">
+        <parent link="base_footprint"/>
+        <child link="base_link" />
+        <origin xyz="0.0 0.0 1.0" rpy="0 0 0"/>
+    </joint>
     <link name="base_link">
         <inertial>
@@ -195,5 +204,4 @@
         <parent link="base_link" />
         <child link="lidar_link" />
-        <axis xyz="0 0 1" />
     </joint>
     <link name="imu_link">

Commit message: make the herminebot to navigate autonomously although badly

File: robot/ros_ws/src/herminebot_description/models/gazebo_plugins.xacro (robot description, xacro)
@@ -28,10 +28,10 @@
             <left_joint>left_wheel_joint</left_joint>
             <right_joint>right_wheel_joint</right_joint>
-            <wheel_separation>0.297</wheel_separation> <!-- Valeur a modifier -->
-            <wheel_diameter>0.06</wheel_diameter> <!-- Valeur a modifier -->
+            <wheel_separation>0.235</wheel_separation>
+            <wheel_diameter>0.06</wheel_diameter>
             <command_topic>cmd_vel</command_topic>
             <!-- Limits -->
-            <max_wheel_torque>200</max_wheel_torque>
-            <max_wheel_acceleration>10.0</max_wheel_acceleration>
+            <max_wheel_torque>20</max_wheel_torque>
+            <max_wheel_acceleration>1.0</max_wheel_acceleration>
             <!-- Output -->
             <odometry_frame>odom</odometry_frame>

File: robot/ros_ws/src/herminebot_description/models/herminebot_core.xacro (robot description, xacro)
@@ -9,21 +9,21 @@
         <parent link="base_footprint"/>
         <child link="base_link" />
-        <origin xyz="0.0 0.0 1.0" rpy="0 0 0"/>
+        <origin xyz="0.0 0.0 0.02" rpy="0 0 0"/>
     </joint>
     <link name="base_link">
         <inertial>
-            <origin xyz="-0.01422 -0.00104 0.1648" rpy="0 0 0" />
+            <origin xyz="-0.00104 0.01422 0.1648" rpy="0 0 0" />
             <mass value="5" />
             <inertia
                 ixx="0.0"
-                ixy="-0.00000060186"
-                ixz="-0.00371774"
+                ixy="0.0"
+                ixz="0.00092280"
                 iyy="0.0"
-                iyz="0.00092280"
+                iyz="0.00371774"
                 izz="0.05153320"
             />
         </inertial>
         <visual>
-            <origin xyz="0 0 0" rpy="-1.5708 0 3.1415" />
+            <origin xyz="0 0 0" rpy="-1.5708 0 1.5708" />
             <geometry>
                 <mesh filename="file://$(find herminebot_description)/meshes/base_link.STL" />
@@ -34,5 +34,5 @@
         </visual>
         <collision>
-            <origin xyz="0 0 0" rpy="-1.5708 0 3.1415" />
+            <origin xyz="0 0 0" rpy="-1.5708 0 1.5708" />
             <geometry>
                 <mesh filename="file://$(find herminebot_description)/meshes/base_link.STL" />
@@ -42,17 +42,17 @@
     <link name="left_wheel_link">
         <inertial>
-            <origin xyz="0.0225 -4.8117E-16 0" rpy="0 0 0" />
+            <origin xyz="0 0 -0.0225" rpy="0 0 0" />
             <mass value="0.2" />
             <inertia
-                ixx="4.2948E-05"
-                ixy="-6.9997E-22"
-                ixz="2.4627E-21"
+                ixx="3.147E-05"
+                ixy="0"
+                ixz="0"
                 iyy="3.147E-05"
-                iyz="-2.647E-23"
-                izz="3.147E-05"
+                iyz="0"
+                izz="4.2948E-05"
             />
         </inertial>
         <visual>
-            <origin xyz="0 0 0" rpy="0 0 0" />
+            <origin xyz="0 0 0" rpy="0 1.5708 0" />
             <geometry>
                 <mesh filename="file://$(find herminebot_description)/meshes/left_wheel_link.STL" />
@@ -63,5 +63,5 @@
         </visual>
         <collision>
-            <origin xyz="0 0 0" rpy="0 0 0" />
+            <origin xyz="0 0 0" rpy="0 1.5708 0" />
             <geometry>
                 <mesh filename="file://$(find herminebot_description)/meshes/left_wheel_link.STL" />
@@ -70,25 +70,24 @@
     </link>
     <joint name="left_wheel_joint" type="continuous">
-        <origin xyz="0.1175 0 0.02" rpy="1.564 0.0 3.1416" />
+        <origin xyz="0 0.1175 0.02" rpy="1.564 0.0 3.1416" />
         <parent link="base_link" />
         <child link="left_wheel_link" />
-        <axis xyz="1 0 0" />
-        <limit lower="0" upper="0" effort="0" velocity="0" />
+        <axis xyz="0 0 1" />
     </joint>
     <link name="right_wheel_link">
         <inertial>
-            <origin xyz="0.0225 -4.1842E-16 3.4694E-18" rpy="0 0 0" />
+            <origin xyz="0 0 -0.0225" rpy="0 0 0" />
             <mass value="0.2" />
             <inertia
-                ixx="4.2948E-05"
-                ixy="3.0585E-20"
-                ixz="1.8206E-21"
+                ixx="3.147E-05"
+                ixy="0"
+                ixz="0"
                 iyy="3.147E-05"
-                iyz="1.6411E-21"
-                izz="3.147E-05"
+                iyz="0"
+                izz="4.2948E-05"
             />
         </inertial>
         <visual>
-            <origin xyz="-0.045 0 0" rpy="0 0 0" />
+            <origin xyz="0 0 0.045" rpy="0 1.5708 0" />
             <geometry>
                 <mesh filename="file://$(find herminebot_description)/meshes/right_wheel_link.STL" />
@@ -99,5 +98,5 @@
         </visual>
         <collision>
-            <origin xyz="-0.045 0 0" rpy="0 0 0" />
+            <origin xyz="0 0 0.045" rpy="0 1.5708 0" />
             <geometry>
                 <mesh filename="file://$(find herminebot_description)/meshes/right_wheel_link.STL" />
@@ -106,80 +105,8 @@
     </link>
     <joint name="right_wheel_joint" type="continuous">
-        <origin xyz="-0.1175 0 0.02" rpy="1.564 0.0 3.1416" />
+        <origin xyz="0 -0.1175 0.02" rpy="1.564 0.0 3.1416" />
         <parent link="base_link" />
         <child link="right_wheel_link" />
-        <axis xyz="1 0 0" />
-    </joint>
-    <link name="gripper_left_link">
-        <inertial>
-            <origin xyz="0.0069271 -0.002 -0.0058473" rpy="0 0 0" />
-            <mass value="0.034943" />
-            <inertia
-                ixx="2.1133E-05"
-                ixy="-1.9167E-06"
-                ixz="2.8841E-06"
-                iyy="1.4367E-05"
-                iyz="6.2513E-06"
-                izz="1.2673E-05"
-            />
-        </inertial>
-        <visual>
-            <origin xyz="0 0 0" rpy="1.5708 3.1415 0" />
-            <geometry>
-                <mesh filename="file://$(find herminebot_description)/meshes/gripper_left_link.STL" />
-            </geometry>
-            <material name="">
-                <color rgba="1 0 0 1" />
-            </material>
-        </visual>
-        <collision>
-            <origin xyz="0 0 0" rpy="0 0 0" />
-            <geometry>
-                <mesh filename="file://$(find herminebot_description)/meshes/gripper_left_link.STL" />
-            </geometry>
-        </collision>
-    </link>
-    <joint name="gripper_left_joint" type="prismatic">
-        <origin xyz="0.085 0.105 0.0" rpy="-3.1416 0 0" />
-        <parent link="base_link" />
-        <child link="gripper_left_link" />
-        <axis xyz="0 0 -1" />
-        <limit lower="0.05" upper="0.25" effort="100" velocity="1" />
-    </joint>
-    <link name="gripper_right_link">
-        <inertial>
-            <origin xyz="0.0069271 0.0030988 0.00025266" rpy="0 0 0" />
-            <mass value="0.034943" />
-            <inertia
-                ixx="2.1133E-05"
-                ixy="-1.9167E-06"
-                ixz="2.8841E-06"
-                iyy="1.4367E-05"
-                iyz="6.2513E-06"
-                izz="1.2673E-05"
-            />
-        </inertial>
-        <visual>
-            <origin xyz="0 0 0" rpy="1.5708 3.1415 0" />
-            <geometry>
-                <mesh filename="file://$(find herminebot_description)/meshes/gripper_right_link.STL" />
-            </geometry>
-            <material name="">
-                <color rgba="0.79216 0.81961 0.93333 1" />
-            </material>
-        </visual>
-        <collision>
-            <origin xyz="0 0 0" rpy="0 0 0" />
-            <geometry>
-                <mesh filename="file://$(find herminebot_description)/meshes/gripper_right_link.STL" />
-            </geometry>
-        </collision>
-    </link>
-    <joint name="gripper_right_joint" type="prismatic">
-        <origin xyz="-0.085 0.105 0.0" rpy="-3.1416 0 0" />
-        <parent link="base_link" />
-        <child link="gripper_right_link" />
-        <axis xyz="0 0 -1" />
-        <limit lower="0.05" upper="0.25" effort="100" velocity="1" />
+        <axis xyz="0 0 1" />
     </joint>
     <link name="lidar_link">
@@ -219,5 +146,5 @@
         </inertial>
         <visual>
-            <origin xyz="0 0 0" rpy="0 0 0" />
+            <origin xyz="0 0 0" rpy="0 0 1.5708" />
             <geometry>
                 <mesh filename="file://$(find herminebot_description)/meshes/imu_link.STL" />
@@ -228,5 +155,5 @@
         </visual>
         <collision>
-            <origin xyz="0 0 0" rpy="0 0 0" />
+            <origin xyz="0 0 0" rpy="0 0 1.5708" />
             <geometry>
                 <mesh filename="file://$(find herminebot_description)/meshes/imu_link.STL" />
@@ -235,5 +162,5 @@
     </link>
     <joint name="imu_joint" type="fixed">
-        <origin xyz="-0.0032751 0.05685 0.029" rpy="0 0 0" />
+        <origin xyz="0.05685 -0.0032751 0.029" rpy="0 0 0" />
         <parent link="base_link" />
         <child link="imu_link" />
