Commit message: refactor herminebot model for gazebo so inertial matrix are not necessary in gazebo.
This allow the robot to move straight and rotate perfectly on itself

File: robot/ros_ws/src/herminebot_description/models/herminebot.urdf (robot description, URDF)
Before this commit: robot herminebot, 0 links, 0 joints
Links:
- added link base_footprint
- added link base_link, mass 5; collision mesh filename=file://$(find herminebot_description)/meshes/base_link.STL; visual mesh filename=file://$(find herminebot_description)/meshes/base_link.STL
- added link imu_link, mass 0.00374; collision mesh filename=file://$(find herminebot_description)/meshes/imu_link.STL; visual mesh filename=file://$(find herminebot_description)/meshes/imu_link.STL
- added link left_wheel_link, mass 0.2; collision mesh filename=file://$(find herminebot_description)/meshes/left_wheel_lin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; visual mesh filename=file://$(find herminebot_description)/meshes/left_wheel_lin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
- added link lidar_link; collision mesh filename=file://$(find herminebot_description)/meshes/lidar_link.STL; visual mesh filename=file://$(find herminebot_description)/meshes/lidar_link.STL
- added link right_wheel_link, mass 0.2; collision mesh filename=file://$(find herminebot_description)/meshes/right_wheel_li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; visual mesh filename=file://$(find herminebot_description)/meshes/right_wheel_li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
Joints:
- added joint base_joint: type fixed, parent base_footprint, child base_link, origin xyz=0.0 0.0 0.02 rpy=0 0 0
- added joint imu_joint: type fixed, parent base_link, child imu_link, origin xyz=0.05685 -0.0032751 0.029 rpy=0 0 0, axis 0 0 0
- added joint left_wheel_joint: type continuous, parent base_link, child left_wheel_link, origin xyz=0 0.1175 0.02 rpy=1.564 0.0 3.1416, axis 0 0 1
- added joint lidar_joint: type fixed, parent base_link, child lidar_link, origin xyz=0 0 0.383 rpy=0 0 -3.1416
- added joint right_wheel_joint: type continuous, parent base_link, child right_wheel_link, origin xyz=0 -0.1175 0.02 rpy=1.564 0.0 3.1416, axis 0 0 1

Commit message: rebuild the herminebot model

File: robot/ros_ws/src/herminebot_description/models/herminebot.urdf (robot description, URDF)
Before this commit: robot herminebot, 6 links, 5 joints
Links:
- removed link left_wheel_link
- removed link right_wheel_link
- link base_link: geometry collision mesh filename=package://herminebot_gazebo/models/herminebot/meshes/base_c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; visual mesh filename=package://herminebot_gazebo/models/herminebot/meshes/base_v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
- link imu_link: mass 0.00374 -> None; geometry 
- link lidar_link: geometry collision cylinder length=0.118 radius=0.05; visual mesh filename=package://herminebot_gazebo/models/herminebot/meshes/lidar.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
Joints:
- removed joint left_wheel_joint
- removed joint right_wheel_joint
- joint base_joint: origin xyz=0.0 0.0 0.02 rpy=0 0 0 -> xyz=0.0 0.0 0.0 rpy=0 0 0
- joint imu_joint: axis 0 0 0 -> (none); origin xyz=0.05685 -0.0032751 0.029 rpy=0 0 0 -> xyz=0 0 0.029 rpy=0 0 0
- joint lidar_joint: origin xyz=0 0 0.383 rpy=0 0 -3.1416 -> xyz=0 0 0 rpy=0 0 0

Commit message: add imu visual

File: robot/ros_ws/src/herminebot_description/models/herminebot.urdf (robot description, URDF)
Before this commit: robot herminebot, 4 links, 3 joints
Links:
- link imu_link: geometry collision box size=0.019 0.027 0.03; visual box size=0.019 0.027 0.003
Joints:
- joint imu_joint: origin xyz=0 0 0.029 rpy=0 0 0 -> xyz=0 0 0 rpy=0 0 0
