Commit message: refactor herminebot model
- Set a specific name for each herminebot model

Why?
It allows to have multiple models

File: robot/ros_ws/src/herminebot_description/models/herminebot_diff.urdf (robot description, URDF)
Before this commit: robot herminebot, 4 links, 3 joints
Links:
- link base_link: geometry collision mesh filename=package://herminebot_gazebo/models/herminebot_diff/meshes/b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; visual mesh filename=package://herminebot_gazebo/models/herminebot_diff/meshes/b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
- link lidar_link: geometry collision cylinder length=0.118 radius=0.05; visual mesh filename=package://herminebot_gazebo/models/herminebot_diff/meshes/l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
