Commit message: add lidar and imu so the robot can navigate
NOTE: The robot slips a lot so it is difficult to have a correct navigation

File: robot/ros_ws/src/herminebot_description/models/herminebot_omni.urdf (robot description, URDF)
Before this commit: robot herminebot_diff, 2 links, 1 joints
Links:
- added link imu_link; collision box size=0.019 0.027 0.03; visual box size=0.019 0.027 0.003
- added link lidar_link; collision cylinder length=0.118 radius=0.05; visual mesh filename=package://herminebot_gazebo/models/herminebot_omni/meshes/l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
Joints:
- added joint imu_joint: type fixed, parent base_link, child imu_link, origin xyz=0 0 0 rpy=0 0 0
- added joint lidar_joint: type fixed, parent base_link, child lidar_link, origin xyz=0 0 0 rpy=0 0 0
